File: pcb/gamepad/gamepad.kicad_sch (KiCad schematic)
At the start: 26 parts, among them J1 PiZero2W, SW1 SW_DIP_x04, SW10 Button1, SW11 RotaryEncoder_Switch, SW12 RotaryEncoder_Switch, SW13 RotaryEncoder_Switch, SW2 RotaryEncoder_Switch, SW3 Button1, SW4 Button1, SW5 Button1, SW6 Button1, SW7 Button1, SW8 Button1, SW9 Button1, U1 THB001P, U2 MCP3008, U3 MCP3008, U4 MCP23017_SP

Commit message: wip pcb
Parts:
- removed SW1: SW_DIP_x04, symbol Switch:SW_DIP_x04
- removed SW10, SW7, SW8, SW9: Button1, symbol Switch:SW_Push
- removed U4: MCP23017_SP, Package_DIP:DIP-28_W7.62mm, symbol Interface_Expansion:MCP23017_SP
- added A1: Arduino_Nano_v3.x, Module:Arduino_Nano, symbol MCU_Module:Arduino_Nano_v3.x
- added J1: Arduino Analogs, Connector_PinSocket_2.54mm:PinSocket_1x05_P2.54mm_Vertical, symbol Connector:Conn_01x06_Pin
- added J3: SPI0, Connector_PinSocket_2.54mm:PinSocket_1x05_P2.54mm_Vertical, symbol Connector:Conn_01x05_Pin
- added R1, R10, R11, R12, R13, R14, R15, R16, R17, R18, R2, R3, R4, R5, R6, R7, R8, R9: R10K, Resistor_SMD:R_1206_3216Metric_Pad1.30x1.75mm_HandSolder, symbol Device:R
- added U2: JOY1, THB001P:CNK_THB001P, symbol THB001P:THB001P
- J2: renamed from J1; footprint (none) -> Connector_PinSocket_2.54mm:PinSocket_2x20_P2.54mm_Vertical
- RV1: value J1-HOR -> LIN1; footprint (none) -> Potentiometer_THT:Potentiometer_Bourns_PTA6043_Single_Slide
- RV2: value J1-VERT -> LIN2; footprint (none) -> Potentiometer_THT:Potentiometer_Bourns_PTA6043_Single_Slide
- RV3: value J2-HOR -> LIN3; footprint (none) -> Potentiometer_THT:Potentiometer_Bourns_PTA4543_Single_Slide
- RV4: value J2-VERT -> LIN4; footprint (none) -> Potentiometer_THT:Potentiometer_Bourns_PTA4543_Single_Slide
- RV5: footprint (none) -> Potentiometer_THT:Potentiometer_Bourns_PTV09A-1_Single_Vertical
- RV6: value ROTARY1 -> ROTARY2; footprint (none) -> Potentiometer_THT:Potentiometer_Bourns_PTV09A-1_Single_Vertical
- RV7: value ROTARY1 -> ROTARY3; footprint (none) -> Potentiometer_THT:Potentiometer_Bourns_PTV09A-1_Single_Vertical
- RV8: value ROTARY1 -> ROTARY4; footprint (none) -> Potentiometer_THT:Potentiometer_Bourns_PTV09A-1_Single_Vertical
- SW1: renamed from SW3; footprint (none) -> Button_Switch_THT:SW_SPST_Omron_B3F-40xx
- SW2: renamed from SW4; value Button1 -> Button2; footprint (none) -> Button_Switch_THT:SW_SPST_Omron_B3F-40xx
- SW3: renamed from SW5; value Button1 -> Button3; footprint (none) -> Button_Switch_THT:SW_SPST_Omron_B3F-40xx
- SW4: renamed from SW6; value Button1 -> Button4; footprint (none) -> Button_Switch_THT:SW_SPST_Omron_B3F-40xx
- SW5: renamed from SW13; value RotaryEncoder_Switch -> Rotary1; footprint (none) -> PEC11R-4215F-S0024:PEC11R-4215F-S0024; symbol Device:RotaryEncoder_Switch -> projectlib:RotaryEncoder_Switch_Fixed
- SW6: renamed from SW11; value RotaryEncoder_Switch -> Rotary2; footprint (none) -> PEC11R-4215F-S0024:PEC11R-4215F-S0024; symbol Device:RotaryEncoder_Switch -> projectlib:RotaryEncoder_Switch_Fixed
- SW7: renamed from SW12; value RotaryEncoder_Switch -> Rotary3; footprint (none) -> PEC11R-4215F-S0024:PEC11R-4215F-S0024; symbol Device:RotaryEncoder_Switch -> projectlib:RotaryEncoder_Switch_Fixed
- SW8: renamed from SW2; value RotaryEncoder_Switch -> Rotary4; footprint (none) -> PEC11R-4215F-S0024:PEC11R-4215F-S0024; symbol Device:RotaryEncoder_Switch -> projectlib:RotaryEncoder_Switch_Fixed
- U1: value THB001P -> JOY2; Check_prices (none) -> https://www.snapeda.com/parts/THB001P/C%2526K/view-part/?re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; Description_1 (none) -> Multi-Directional Thumbstick, 2 Axis, Center Momentary Swit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; DigiKey_Part_Number (none) -> 108-THB001P-ND; MF (none) -> C&K; MP (none) -> THB001P; Package (none) -> None; SnapEDA_Link (none) -> https://www.snapeda.com/parts/THB001P/C%2526K/view-part/?re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
- U3: renamed from U2; footprint (none) -> Package_DIP:CERDIP-16_W7.62mm_SideBrazed_Socket
- U4: renamed from U3; footprint (none) -> Package_DIP:CERDIP-16_W7.62mm_SideBrazed_Socket
Connections:
- net 3V3: now also U1.VR1_3, U1.VR2_3, A1.17 (3V3), U2.VR1_3, U2.VR2_3
- net 5V: now also A1.27 (+5V), A1.30 (VIN)
- net GND: now also SW5.COM (Com), SW6.COM (Com), SW7.COM (Com), SW8.COM (Com), U1.VR1_1, U1.VR2_1, A1.29 (GND), A1.4 (GND), R11.2, R14.2, R17.2, R2.2, R3.2, R4.2, R5.2, R6.2, R8.2, R9.2, U2.VR1_1, U2.VR2_1
- net at U4.1 (CH0): now also U2.VR1_2
- net at U4.2 (CH1): now also U2.VR2_2
- net at U4.3 (CH2): now also U1.VR2_2
- net at U4.4 (CH3): now also U1.VR1_2
- net BTN4: now reaches SW4.1
- net BTN4: now also J2.22 (GPIO25)
- net at SW4.2: now also R5.1
- net JOY-BTN2: now reaches J2.13 (GPIO27)
- net JOY-BTN2: now also U1.C, U1.D
- net BTN1: now reaches J2.15 (GPIO22)
- net BTN1: now also SW1.1
- net BTN2: now reaches J2.16 (GPIO23)
- net BTN2: now also SW2.1
- net BTN3: now reaches J2.18 (GPIO24)
- net BTN3: now also SW3.1
- net at J2.19 (MOSI0/GPIO10): now also J3.2 (Pin_2)
- net at J2.21 (MISO0/GPIO9): now also J3.3 (Pin_3)
- net at J2.23 (SCLK0/GPIO11): now also J3.1 (Pin_1)
- net at J2.24 (~{CE0}/GPIO8): now also J3.4 (Pin_4)
- net at J2.26 (~{CE1}/GPIO7): now also J3.5 (Pin_5)
- net RE-SW3: now reaches J2.29 (GCLK1/GPIO5)
- net RE-SW3: now also SW6.1
- net at J2.3 (SDA/GPIO2): now also A1.23 (A4)
- net RE-SW2: now reaches J2.31 (GCLK2/GPIO6)
- net RE-SW2: now also SW7.1
- net RE-SW1: now reaches J2.32 (PWM0/GPIO12)
- net RE-SW1: now also SW8.1
- net JOY-BTN1: now reaches J2.37 (GPIO26)
- net JOY-BTN1: now also U2.C, U2.D
- net at J2.5 (SCL/GPIO3): now also A1.24 (A5)
- net RE-SW4: now reaches J2.7 (GCLK0/GPIO4)
- net RE-SW4: now also SW5.1
- net at SW3.2: now also R4.1
- net at SW5.A: now also R1.2
- net at SW5.B: now also R7.1
- net at SW8.A: now also R16.2
- net at SW8.B: now also R18.1
- net at SW1.2: now also R2.1
- net at SW7.A: now also R13.2
- net at SW7.B: now also R15.1
- net at SW6.A: now also R10.2
- net at SW6.B: now also R12.1
- net at SW2.2: now also R3.1
- net at U1.A: now also U1.B, R9.1
- new net: R8.1, U2.A, U2.B
- new net: A1.11 (D8), R7.2
- new net: R6.1, SW5.2
- new net: A1.10 (D7), R10.1
- new net: A1.12 (D9), R1.1
- new net: A1.19 (A0), J1.6 (Pin_6)
- new net: A1.20 (A1), J1.5 (Pin_5)
- new net: A1.21 (A2), J1.4 (Pin_4)
- new net: A1.22 (A3), J1.3 (Pin_3)
- new net: A1.25 (A6), J1.2 (Pin_2)
- new net: A1.26 (A7), J1.1 (Pin_1)
- new net: A1.5 (D2), R18.2
- new net: A1.6 (D3), R16.1
- new net: A1.7 (D4), R15.2
- new net: A1.8 (D5), R13.1
- new net: A1.9 (D6), R12.2
- new net: R11.1, SW6.2
- new net: R17.1, SW8.2
- new net: R14.1, SW7.2
- no-connect marks 0 -> 14
Other:
- moved on the sheet: J2, RV1, RV2, RV3, RV4, RV5, RV6, RV7, RV8, SW1, SW2, SW3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
