File: pcb/gamepadv2/gamepad.kicad_sch (KiCad schematic)
At the start: 29 parts, among them J1 PowerConnector, J2 PiZero2W, SW1 Button1, SW2 Button2, SW3 Button3, SW4 Button4, SW5 Button5, SW6 Button6, SW7 Button7, SW8 Button8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

Commit message: wip
Parts:
- RV3, RV4: footprint Potentiometer_THT:Potentiometer_Bourns_PTA4543_Single_Slide -> Potentiometer_THT:Potentiometer_Bourns_PTA6043_Single_Slide
Changed lines of the file:
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@@
 			)
 		)
-		(property "Footprint" "Potentiometer_THT:Potentiometer_Bourns_PTA4543_Single_Slide"
+		(property "Footprint" "Potentiometer_THT:Potentiometer_Bourns_PTA6043_Single_Slide"
 			(at 49.53 54.61 0)
 			(effects
@@
 			)
 		)
-		(property "Footprint" "Potentiometer_THT:Potentiometer_Bourns_PTA4543_Single_Slide"
+		(property "Footprint" "Potentiometer_THT:Potentiometer_Bourns_PTA6043_Single_Slide"
 			(at 49.53 45.72 0)
 			(effects
